Commit message: Add gazebo support

File: urdf/robot.urdf (robot description, URDF)
Before this commit: robot abb_arm, 8 links, 7 joints
Links:
- link irb4600_60kg_205_base_cad_rev05_v1: geometry collision mesh filename=file://$(find abb_arm_description)/abb_arm/assets/irb4600_6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; visual mesh filename=file://$(find abb_arm_description)/abb_arm/assets/irb4600_6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
- link irb4600_60kg_205_link1_cad_rev04_v1: geometry collision mesh filename=file://$(find abb_arm_description)/abb_arm/assets/irb4600_6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; visual mesh filename=file://$(find abb_arm_description)/abb_arm/assets/irb4600_6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
- link irb4600_60kg_205_link2_cad_rev04_v1: geometry collision mesh filename=file://$(find abb_arm_description)/abb_arm/assets/irb4600_6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; visual mesh filename=file://$(find abb_arm_description)/abb_arm/assets/irb4600_6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
- link irb4600_60kg_205_link3_cad_rev04_v1: geometry collision mesh filename=file://$(find abb_arm_description)/abb_arm/assets/irb4600_6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; visual mesh filename=file://$(find abb_arm_description)/abb_arm/assets/irb4600_6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
- link irb4600_60kg_205_link4_cad_rev04_v1: geometry collision mesh filename=file://$(find abb_arm_description)/abb_arm/assets/irb4600_6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; visual mesh filename=file://$(find abb_arm_description)/abb_arm/assets/irb4600_6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
- link irb4600_60kg_205_link5_cad_rev04_v1: geometry collision mesh filename=file://$(find abb_arm_description)/abb_arm/assets/irb4600_6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; visual mesh filename=file://$(find abb_arm_description)/abb_arm/assets/irb4600_6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
- link irb4600_60kg_205_link6_cad_rev04_v1: geometry collision mesh filename=file://$(find abb_arm_description)/abb_arm/assets/irb4600_6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; collision mesh filename=file://$(find abb_arm_description)/abb_arm/assets/polisher.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
Joints:
- joint base_joint: origin xyz=0 0 0 rpy=0 0 0 -> xyz=0 0 0.5 rpy=0 0 0
