Commit message: Successfully spawn arm in gazebo

File: urdf/abb.xacro (robot description, xacro)
@@ -211,5 +211,5 @@
     <child link="irb4600_60kg_205_link6_cad_rev04_v1"/>
     <axis xyz="0 0 1"/>
-    <limit effort="10" velocity="10" lower="-3.141592653589793" upper="3.141592653589793"/>
+    <limit effort="1000" velocity="10" lower="-3.141592653589793" upper="3.141592653589793"/>
   </joint>
   <!-- Joint from irb4600_60kg_205_link4_cad_rev04_v1 to irb4600_60kg_205_link5_cad_rev04_v1 -->
@@ -219,5 +219,5 @@
     <child link="irb4600_60kg_205_link5_cad_rev04_v1"/>
     <axis xyz="0 0 1"/>
-    <limit effort="10" velocity="10" lower="-3.141592653589793" upper="3.141592653589793"/>
+    <limit effort="1000" velocity="10" lower="-3.141592653589793" upper="3.141592653589793"/>
   </joint>
   <!-- Joint from irb4600_60kg_205_link3_cad_rev04_v1 to irb4600_60kg_205_link4_cad_rev04_v1 -->
@@ -227,5 +227,5 @@
     <child link="irb4600_60kg_205_link4_cad_rev04_v1"/>
     <axis xyz="0 0 1"/>
-    <limit effort="10" velocity="10" lower="-3.141592653589793" upper="3.141592653589793"/>
+    <limit effort="1000" velocity="10" lower="-3.141592653589793" upper="3.141592653589793"/>
   </joint>
   <!-- Joint from irb4600_60kg_205_link2_cad_rev04_v1 to irb4600_60kg_205_link3_cad_rev04_v1 -->
@@ -235,5 +235,5 @@
     <child link="irb4600_60kg_205_link3_cad_rev04_v1"/>
     <axis xyz="0 0 1"/>
-    <limit effort="10" velocity="10" lower="-3.141592653589793" upper="3.141592653589793"/>
+    <limit effort="1000" velocity="10" lower="-3.141592653589793" upper="3.141592653589793"/>
   </joint>
   <!-- Joint from irb4600_60kg_205_link1_cad_rev04_v1 to irb4600_60kg_205_link2_cad_rev04_v1 -->
@@ -243,5 +243,5 @@
     <child link="irb4600_60kg_205_link2_cad_rev04_v1"/>
     <axis xyz="0 0 1"/>
-    <limit effort="10" velocity="10" lower="-3.141592653589793" upper="3.141592653589793"/>
+    <limit effort="1000" velocity="10" lower="-3.141592653589793" upper="3.141592653589793"/>
   </joint>
   <!-- Joint from irb4600_60kg_205_base_cad_rev05_v1 to irb4600_60kg_205_link1_cad_rev04_v1 -->
@@ -251,5 +251,5 @@
     <child link="irb4600_60kg_205_link1_cad_rev04_v1"/>
     <axis xyz="0 0 1"/>
-    <limit effort="10" velocity="10" lower="-3.141592653589793" upper="3.141592653589793"/>
+    <limit effort="1000" velocity="10" lower="-3.141592653589793" upper="3.141592653589793"/>
   </joint>
   <!-- Joint from base_link to base_cad -->

File: urdf/robot.urdf.xacro (robot description, xacro)
@@ -3,3 +3,5 @@
     <!-- Include abb arm -->
     <xacro:include filename="$(find abb_arm_description)/urdf/abb.xacro"/>
+    <!-- Include ros2_control -->
+    <xacro:include filename="$(find abb_arm_description)/urdf/abb_arm.ros2_control.xacro"/>
 </robot>

Commit message: Add platform to robot

File: urdf/abb.xacro (robot description, xacro)
@@ -254,7 +254,7 @@
   </joint>
   <!-- Joint from base_link to base_cad -->
-  <joint name="base_joint" type="fixed">
-    <origin xyz="0 0 0.5" rpy="0 0 0"/>
-    <parent link="base_link"/>
+  <joint name="chassis_arm_base_joint" type="fixed">
+    <origin xyz="0.3 0 0.65" rpy="0 0 0"/>
+    <parent link="chassis"/>
     <child link="irb4600_60kg_205_base_cad_rev05_v1"/>
   </joint>

File: urdf/robot.urdf.xacro (robot description, xacro)
@@ -1,4 +1,8 @@
 <?xml version="1.0"?>
 <robot xmlns:xacro="http://www.ros.org/wiki/xacro" name="abb_arm">
+    <!-- Include inertial macros -->
+    <xacro:include filename="$(find abb_arm_description)/urdf/inertial_macros.xacro"/>
+    <!-- Include platform -->
+    <xacro:include filename="$(find abb_arm_description)/urdf/platform.xacro"/>
     <!-- Include abb arm -->
     <xacro:include filename="$(find abb_arm_description)/urdf/abb.xacro"/>
