Commit message: Fix origin error

File: urdf/major_components.xacro (robot description, xacro)
@@ -158,5 +158,5 @@
     <parent link="base_link"/>
     <child link="base_plate__mild_steel"/>
-    <origin xyz="-0.295151 0.0518164 0.226115" rpy="0 0 0"/>
+    <origin xyz="0 0 0" rpy="0 0 0"/>
   </joint>
 </robot>

Commit message: Add rough mir1350 platform

File: urdf/major_components.xacro (robot description, xacro)
@@ -158,5 +158,5 @@
     <parent link="base_link"/>
     <child link="base_plate__mild_steel"/>
-    <origin xyz="0 0 0" rpy="0 0 0"/>
+    <origin xyz="0 0 0.03" rpy="0 0 0"/>
   </joint>
 </robot>

File: urdf/robot.urdf.xacro (robot description, xacro)
@@ -1,4 +1,6 @@
 <?xml version="1.0"?>
 <robot xmlns:xacro="http://www.ros.org/wiki/xacro" name="abb_arm">
+    <!-- Include color macros -->
+    <xacro:include filename="$(find abb_arm_description)/urdf/colours.xacro"/>
     <!-- Include inertial macros -->
     <xacro:include filename="$(find abb_arm_description)/urdf/inertial_macros.xacro"/>
@@ -10,6 +12,9 @@
     <xacro:include filename="$(find abb_arm_description)/urdf/major_components.xacro"/>
     <!-- Include mir platform -->
-    <xacro:include filename="$(find abb_arm_description)/urdf/mir_platform.xacro"/>
+    <!-- <xacro:include filename="$(find abb_arm_description)/urdf/mir_platform.xacro"/> -->
+    <xacro:include filename="$(find abb_arm_description)/urdf/mir1350_rough.xacro"/>
     <!-- Include ros2_control -->
-    <xacro:include filename="$(find abb_arm_description)/urdf/abb_arm.ros2_control.xacro"/>
+    <xacro:include filename="$(find abb_arm_description)/urdf/ros2_control.xacro"/>
+    <!-- Include gazebo plugins -->
+    <xacro:include filename="$(find abb_arm_description)/urdf/gazebo_control.xacro"/>
 </robot>

File: urdf/ros2_control.xacro (robot description, xacro)
@@ -5,4 +5,5 @@
             <plugin>gz_ros2_control/GazeboSimSystem</plugin>
         </hardware>
+        <!-- ABB Arm -->
         <joint name="joint1">
             <command_interface name="position"/>
@@ -47,4 +48,21 @@
             <state_interface name="velocity"/>
         </joint>
+        <!-- MiR Robot -->
+        <joint name="left_wheel_joint">
+            <command_interface name="velocity">
+                <param name="min">-10</param>
+                <param name="max">10</param>
+            </command_interface>
+            <state_interface name="position"/>
+            <state_interface name="velocity"/>
+        </joint>
+        <joint name="right_wheel_joint">
+            <command_interface name="velocity">
+                <param name="min">-10</param>
+                <param name="max">10</param>
+            </command_interface>
+            <state_interface name="position"/>
+            <state_interface name="velocity"/>
+        </joint>
     </ros2_control>
     <gazebo>
