Commit message: Add control to mir robot rough

File: urdf/mir1350_rough.xacro (robot description, xacro)
@@ -38,4 +38,5 @@
         <origin xyz="0 0.475 -0.25" rpy="-${pi/2} 0 0"/>
         <axis xyz="0 0 1"/>
+        <limit effort="100" velocity="10"/>
     </joint>
     <link name="left_wheel">
@@ -61,4 +62,5 @@
         <origin xyz="0 -0.475 -0.25" rpy="${pi/2} 0 0"/>
         <axis xyz="0 0 -1"/>
+        <limit effort="100" velocity="10"/>
     </joint>
     <link name="right_wheel">

File: urdf/robot.urdf.xacro (robot description, xacro)
@@ -1,4 +1,30 @@
 <?xml version="1.0"?>
 <robot xmlns:xacro="http://www.ros.org/wiki/xacro" name="abb_arm">
+    <gazebo>
+        <plugin name="gz::sim::systems::DiffDrive" filename="gz-sim-diff-drive-system">
+            <!-- Wheel Information -->
+            <left_joint>left_wheel_joint</left_joint>
+            <right_joint>right_wheel_joint</right_joint>
+            <wheel_separation>1.23</wheel_separation>
+            <wheel_radius>0.05</wheel_radius>
+            <!-- Limits -->
+            <max_linear_acceleration>0.66</max_linear_acceleration>
+            <!-- Input -->
+            <topic>/cmd_vel</topic>
+            <!-- Output -->
+            <frame_id>odom</frame_id>
+            <child_frame_id>base_link</child_frame_id>
+            <odom_topic>/odom</odom_topic>
+            <odom_publisher_frequency>100</odom_publisher_frequency>
+            <tf_topic>/tf</tf_topic>
+        </plugin>
+        <plugin name="gz::sim::systems::JointStatePublisher" filename="gz-sim-joint-state-publisher-system">
+            <topic>/joint_states</topic>
+            <joint_name>left_wheel_joint</joint_name>
+            <joint_name>right_wheel_joint</joint_name>
+        </plugin>
+    </gazebo>
+    <!-- Include gazebo plugins -->
+    <!-- <xacro:include filename="$(find abb_arm_description)/urdf/gazebo_control.xacro"/> -->
     <!-- Include color macros -->
     <xacro:include filename="$(find abb_arm_description)/urdf/colours.xacro"/>
@@ -16,5 +42,3 @@
     <!-- Include ros2_control -->
     <xacro:include filename="$(find abb_arm_description)/urdf/ros2_control.xacro"/>
-    <!-- Include gazebo plugins -->
-    <xacro:include filename="$(find abb_arm_description)/urdf/gazebo_control.xacro"/>
 </robot>
