Commit message: Reformat abb_arm files

File: urdf/abb_arm.xacro (robot description, xacro)
@@ -16,5 +16,5 @@
       <origin xyz="-0.223542 -0.043641 -0.379314" rpy="0.00762494 -0.0869335 -0.0875981"/>
       <geometry>
-        <mesh filename="file://$(find abb_arm_description)/abb_arm/assets/irb4600_60kg_205_base_cad_rev05_v1.stl"/>
+        <mesh filename="file://$(find abb_arm_description)/assets/abb_arm/irb4600_60kg_205_base_cad_rev05_v1.stl"/>
       </geometry>
       <material name="irb4600_60kg_205_base_cad_rev05_v1_material">
@@ -25,5 +25,5 @@
       <origin xyz="-0.223542 -0.043641 -0.379314" rpy="0.00762494 -0.0869335 -0.0875981"/>
       <geometry>
-        <mesh filename="file://$(find abb_arm_description)/abb_arm/assets/irb4600_60kg_205_base_cad_rev05_v1.stl"/>
+        <mesh filename="file://$(find abb_arm_description)/assets/abb_arm/irb4600_60kg_205_base_cad_rev05_v1.stl"/>
       </geometry>
     </collision>
@@ -40,5 +40,5 @@
       <origin xyz="4.32987e-15 7.77156e-16 0.1595" rpy="-3.14159 2.77556e-17 -1.09504e-17"/>
       <geometry>
-        <mesh filename="file://$(find abb_arm_description)/abb_arm/assets/irb4600_60kg_205_link1_cad_rev04_v1.stl"/>
+        <mesh filename="file://$(find abb_arm_description)/assets/abb_arm/irb4600_60kg_205_link1_cad_rev04_v1.stl"/>
       </geometry>
       <material name="irb4600_60kg_205_link1_cad_rev04_v1_material">
@@ -49,5 +49,5 @@
       <origin xyz="4.32987e-15 7.77156e-16 0.1595" rpy="-3.14159 2.77556e-17 -1.09504e-17"/>
       <geometry>
-        <mesh filename="file://$(find abb_arm_description)/abb_arm/assets/irb4600_60kg_205_link1_cad_rev04_v1.stl"/>
+        <mesh filename="file://$(find abb_arm_description)/assets/abb_arm/irb4600_60kg_205_link1_cad_rev04_v1.stl"/>
       </geometry>
     </collision>
@@ -64,5 +64,5 @@
       <origin xyz="-0.175 0.495 0.1225" rpy="1.5708 -3.41524e-17 -1.38778e-17"/>
       <geometry>
-        <mesh filename="file://$(find abb_arm_description)/abb_arm/assets/irb4600_60kg_205_link2_cad_rev04_v1.stl"/>
+        <mesh filename="file://$(find abb_arm_description)/assets/abb_arm/irb4600_60kg_205_link2_cad_rev04_v1.stl"/>
       </geometry>
       <material name="irb4600_60kg_205_link2_cad_rev04_v1_material">
@@ -73,5 +73,5 @@
       <origin xyz="-0.175 0.495 0.1225" rpy="1.5708 -3.41524e-17 -1.38778e-17"/>
       <geometry>
-        <mesh filename="file://$(find abb_arm_description)/abb_arm/assets/irb4600_60kg_205_link2_cad_rev04_v1.stl"/>
+        <mesh filename="file://$(find abb_arm_description)/assets/abb_arm/irb4600_60kg_205_link2_cad_rev04_v1.stl"/>
       </geometry>
     </collision>
@@ -88,5 +88,5 @@
       <origin xyz="-0.175 -1.395 -0.1492" rpy="-1.5708 3.84892e-17 -1.38778e-17"/>
       <geometry>
-        <mesh filename="file://$(find abb_arm_description)/abb_arm/assets/irb4600_60kg_205_link3_cad_rev04_v1.stl"/>
+        <mesh filename="file://$(find abb_arm_description)/assets/abb_arm/irb4600_60kg_205_link3_cad_rev04_v1.stl"/>
       </geometry>
       <material name="irb4600_60kg_205_link3_cad_rev04_v1_material">
@@ -97,5 +97,5 @@
       <origin xyz="-0.175 -1.395 -0.1492" rpy="-1.5708 3.84892e-17 -1.38778e-17"/>
       <geometry>
-        <mesh filename="file://$(find abb_arm_description)/abb_arm/assets/irb4600_60kg_205_link3_cad_rev04_v1.stl"/>
+        <mesh filename="file://$(find abb_arm_description)/assets/abb_arm/irb4600_60kg_205_link3_cad_rev04_v1.stl"/>
       </geometry>
     </collision>
@@ -112,5 +112,5 @@
       <origin xyz="-2.08167e-16 1.57 0.5151" rpy="1.5708 1.5708 0"/>
       <geometry>
-        <mesh filename="file://$(find abb_arm_description)/abb_arm/assets/irb4600_60kg_205_link4_cad_rev04_v1.stl"/>
+        <mesh filename="file://$(find abb_arm_description)/assets/abb_arm/irb4600_60kg_205_link4_cad_rev04_v1.stl"/>
       </geometry>
       <material name="irb4600_60kg_205_link4_cad_rev04_v1_material">
@@ -121,5 +121,5 @@
       <origin xyz="-2.08167e-16 1.57 0.5151" rpy="1.5708 1.5708 0"/>
       <geometry>
-        <mesh filename="file://$(find abb_arm_description)/abb_arm/assets/irb4600_60kg_205_link4_cad_rev04_v1.stl"/>
+        <mesh filename="file://$(find abb_arm_description)/assets/abb_arm/irb4600_60kg_205_link4_cad_rev04_v1.stl"/>
       </geometry>
     </collision>
@@ -136,5 +136,5 @@
       <origin xyz="-1.135 -1.57 -0.067" rpy="-1.5708 -3.79471e-18 -1.38778e-17"/>
       <geometry>
-        <mesh filename="file://$(find abb_arm_description)/abb_arm/assets/irb4600_60kg_205_link5_cad_rev04_v1.stl"/>
+        <mesh filename="file://$(find abb_arm_description)/assets/abb_arm/irb4600_60kg_205_link5_cad_rev04_v1.stl"/>
       </geometry>
       <material name="irb4600_60kg_205_link5_cad_rev04_v1_material">
@@ -145,5 +145,5 @@
       <origin xyz="-1.135 -1.57 -0.067" rpy="-1.5708 -3.79471e-18 -1.38778e-17"/>
       <geometry>
-        <mesh filename="file://$(find abb_arm_description)/abb_arm/assets/irb4600_60kg_205_link5_cad_rev04_v1.stl"/>
+        <mesh filename="file://$(find abb_arm_description)/assets/abb_arm/irb4600_60kg_205_link5_cad_rev04_v1.stl"/>
       </geometry>
     </collision>
@@ -160,5 +160,5 @@
       <origin xyz="8.04912e-16 1.5704 1.17" rpy="1.5708 1.5708 0"/>
       <geometry>
-        <mesh filename="file://$(find abb_arm_description)/abb_arm/assets/polisher.stl"/>
+        <mesh filename="file://$(find abb_arm_description)/assets/abb_arm/polisher.stl"/>
       </geometry>
       <material name="polisher_material">
@@ -169,5 +169,5 @@
       <origin xyz="8.04912e-16 1.5704 1.17" rpy="1.5708 1.5708 0"/>
       <geometry>
-        <mesh filename="file://$(find abb_arm_description)/abb_arm/assets/polisher.stl"/>
+        <mesh filename="file://$(find abb_arm_description)/assets/abb_arm/polisher.stl"/>
       </geometry>
     </collision>
@@ -176,5 +176,5 @@
       <origin xyz="1.66533e-16 1.57 1.2" rpy="1.5708 1.5708 0"/>
       <geometry>
-        <mesh filename="file://$(find abb_arm_description)/abb_arm/assets/irb4600_60kg_205_link6_cad_rev04_v1.stl"/>
+        <mesh filename="file://$(find abb_arm_description)/assets/abb_arm/irb4600_60kg_205_link6_cad_rev04_v1.stl"/>
       </geometry>
       <material name="irb4600_60kg_205_link6_cad_rev04_v1_material">
@@ -185,5 +185,5 @@
       <origin xyz="1.66533e-16 1.57 1.2" rpy="1.5708 1.5708 0"/>
       <geometry>
-        <mesh filename="file://$(find abb_arm_description)/abb_arm/assets/irb4600_60kg_205_link6_cad_rev04_v1.stl"/>
+        <mesh filename="file://$(find abb_arm_description)/assets/abb_arm/irb4600_60kg_205_link6_cad_rev04_v1.stl"/>
       </geometry>
     </collision>
@@ -192,5 +192,5 @@
       <origin xyz="7.35523e-16 1.57 1.2" rpy="1.5708 1.5708 0"/>
       <geometry>
-        <mesh filename="file://$(find abb_arm_description)/abb_arm/assets/polisher__2.stl"/>
+        <mesh filename="file://$(find abb_arm_description)/assets/abb_arm/polisher__2.stl"/>
       </geometry>
       <material name="polisher_2_material">
@@ -201,5 +201,5 @@
       <origin xyz="7.35523e-16 1.57 1.2" rpy="1.5708 1.5708 0"/>
       <geometry>
-        <mesh filename="file://$(find abb_arm_description)/abb_arm/assets/polisher__2.stl"/>
+        <mesh filename="file://$(find abb_arm_description)/assets/abb_arm/polisher__2.stl"/>
       </geometry>
     </collision>
@@ -254,8 +254,14 @@
   </joint>
   <!-- Joint from base_link to base_cad -->
-  <joint name="chassis_arm_base_joint" type="fixed">
+  <!-- <joint name="chassis_arm_base_joint" type="fixed">
     <origin xyz="0.3 0 0.65" rpy="0 0 0"/>
     <parent link="chassis"/>
     <child link="irb4600_60kg_205_base_cad_rev05_v1"/>
+  </joint> -->
+  <!-- Joint from base_plate to base_cad -->
+  <joint name="base_plate_base_cad_joint" type="fixed">
+    <origin xyz="0.62 0.08 0.4" rpy="0 0.05 0.1"/>
+    <parent link="base_plate__mild_steel"/>
+    <child link="irb4600_60kg_205_base_cad_rev05_v1"/>
   </joint>
 </robot>

Commit message: Minor tweaks

File: urdf/abb_arm.xacro (robot description, xacro)
@@ -261,5 +261,5 @@
   <!-- Joint from base_plate to base_cad -->
   <joint name="base_plate_base_cad_joint" type="fixed">
-    <origin xyz="0.62 0.08 0.4" rpy="0 0.05 0.1"/>
+    <origin xyz="0.62 0.08 0.391" rpy="0 0.08 0.1"/>
     <parent link="base_plate__mild_steel"/>
     <child link="irb4600_60kg_205_base_cad_rev05_v1"/>

Commit message: Add Moveit capabilities

File: urdf/abb_arm.xacro (robot description, xacro)
@@ -211,5 +211,5 @@
     <child link="irb4600_60kg_205_link6_cad_rev04_v1"/>
     <axis xyz="0 0 1"/>
-    <limit effort="1000" velocity="10" lower="-3.141592653589793" upper="3.141592653589793"/>
+    <limit effort="10000" velocity="10" lower="-3.141592653589793" upper="3.141592653589793"/>
   </joint>
   <!-- Joint from irb4600_60kg_205_link4_cad_rev04_v1 to irb4600_60kg_205_link5_cad_rev04_v1 -->
@@ -219,5 +219,5 @@
     <child link="irb4600_60kg_205_link5_cad_rev04_v1"/>
     <axis xyz="0 0 1"/>
-    <limit effort="1000" velocity="10" lower="-3.141592653589793" upper="3.141592653589793"/>
+    <limit effort="10000" velocity="10" lower="-3.141592653589793" upper="3.141592653589793"/>
   </joint>
   <!-- Joint from irb4600_60kg_205_link3_cad_rev04_v1 to irb4600_60kg_205_link4_cad_rev04_v1 -->
@@ -227,5 +227,5 @@
     <child link="irb4600_60kg_205_link4_cad_rev04_v1"/>
     <axis xyz="0 0 1"/>
-    <limit effort="1000" velocity="10" lower="-3.141592653589793" upper="3.141592653589793"/>
+    <limit effort="10000" velocity="10" lower="-3.141592653589793" upper="3.141592653589793"/>
   </joint>
   <!-- Joint from irb4600_60kg_205_link2_cad_rev04_v1 to irb4600_60kg_205_link3_cad_rev04_v1 -->
@@ -235,5 +235,5 @@
     <child link="irb4600_60kg_205_link3_cad_rev04_v1"/>
     <axis xyz="0 0 1"/>
-    <limit effort="1000" velocity="10" lower="-3.141592653589793" upper="3.141592653589793"/>
+    <limit effort="10000" velocity="10" lower="-3.141592653589793" upper="3.141592653589793"/>
   </joint>
   <!-- Joint from irb4600_60kg_205_link1_cad_rev04_v1 to irb4600_60kg_205_link2_cad_rev04_v1 -->
@@ -243,5 +243,5 @@
     <child link="irb4600_60kg_205_link2_cad_rev04_v1"/>
     <axis xyz="0 0 1"/>
-    <limit effort="1000" velocity="10" lower="-3.141592653589793" upper="3.141592653589793"/>
+    <limit effort="10000" velocity="10" lower="-3.141592653589793" upper="3.141592653589793"/>
   </joint>
   <!-- Joint from irb4600_60kg_205_base_cad_rev05_v1 to irb4600_60kg_205_link1_cad_rev04_v1 -->
@@ -251,5 +251,5 @@
     <child link="irb4600_60kg_205_link1_cad_rev04_v1"/>
     <axis xyz="0 0 1"/>
-    <limit effort="1000" velocity="10" lower="-3.141592653589793" upper="3.141592653589793"/>
+    <limit effort="10000" velocity="10" lower="-3.141592653589793" upper="3.141592653589793"/>
   </joint>
   <!-- Joint from base_link to base_cad -->

File: urdf/ros2_control.xacro (robot description, xacro)
@@ -4,4 +4,5 @@
         <hardware>
             <plugin>gz_ros2_control/GazeboSimSystem</plugin>
+            <!-- <plugin>mock_components/GenericSystem</plugin> -->
         </hardware>
         <!-- ABB Arm -->

Commit message: Add LIDAR to robot

File: urdf/abb_arm.xacro (robot description, xacro)
@@ -3,6 +3,4 @@
 <!-- Onshape document_id f0912ad76048a2e7ed12d76c -->
 <robot xmlns:xacro="http://www.ros.org/wiki/xacro" name="abb_arm">
-  <!-- Base link -->
-  <link name="base_link" />
   <!-- Link irb4600_60kg_205_base_cad_rev05_v1 -->
   <link name="irb4600_60kg_205_base_cad_rev05_v1">

File: urdf/major_components.xacro (robot description, xacro)
@@ -156,7 +156,7 @@
   </link>
   <joint name="base_plate_mild_steel_joint" type="fixed">
-    <parent link="base_link"/>
+    <parent link="chassis"/>
     <child link="base_plate__mild_steel"/>
-    <origin xyz="0 0 0.03" rpy="0 0 0"/>
+    <origin xyz="0 0 0.282" rpy="0 0 0"/>
   </joint>
 </robot>

File: urdf/mir1350_rough.xacro (robot description, xacro)
@@ -1,4 +1,6 @@
 <?xml version="1.0"?>
 <robot xmlns:xacro="http://www.ros.org/wiki/xacro">
+    <!-- Include LIDAR -->
+    <xacro:include filename="$(find abb_arm_description)/urdf/lidar.xacro"/>
     <joint name="base_footprint_joint" type="fixed">
         <parent link="base_link"/>
@@ -12,5 +14,5 @@
         <parent link="base_link"/>
         <child link="chassis"/>
-        <origin xyz="0 0 -0.25"/>
+        <origin xyz="0 0 0"/>
     </joint>
     <link name="chassis">
@@ -36,5 +38,5 @@
         <parent link="base_link"/>
         <child link="left_wheel"/>
-        <origin xyz="0 0.475 -0.25" rpy="-${pi/2} 0 0"/>
+        <origin xyz="0 0.475 0" rpy="-${pi/2} 0 0"/>
         <axis xyz="0 0 1"/>
         <limit effort="100" velocity="10"/>
@@ -60,5 +62,5 @@
         <parent link="base_link"/>
         <child link="right_wheel"/>
-        <origin xyz="0 -0.475 -0.25" rpy="${pi/2} 0 0"/>
+        <origin xyz="0 -0.475 0" rpy="${pi/2} 0 0"/>
         <axis xyz="0 0 -1"/>
         <limit effort="100" velocity="10"/>

File: urdf/robot.urdf.xacro (robot description, xacro)
@@ -25,6 +25,5 @@
         </plugin>
     </gazebo>
-    <!-- Include gazebo plugins -->
-    <!-- <xacro:include filename="$(find abb_arm_description)/urdf/gazebo_control.xacro"/> -->
+    <link name="base_link"/>
     <!-- Include color macros -->
     <xacro:include filename="$(find abb_arm_description)/urdf/colours.xacro"/>
